File: MiniARMBoard.brd (EAGLE design)
At the start: 35.6 x 20.6 mm, 39 parts, among them CN1 J_USB_MICROAB_HIROSE_ZX62-AB-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, IC1 TPD4S014DSQR, IC2 FT234XD-R, U1 LPC1549JBD48, U3 MCP1700T-33, U4 ADR5041, X1 FA238V

Commit message: ICの名前を'IC*'から'U*'に変更
Parts:
- renumbered IC1 to U2, IC2 to U5
